File: snapstone_pcb/redstone_repeater/redstone_repeater.kicad_sch (KiCad schematic)
At the start: 23 parts, among them Q1 MMBFJ270_Analog_Switch, Q2 MMBFJ270_Analog_Switch, SW1 SW_Push, SW2 SW_Push, SW3 SW_Push, SW4 SW_Push, U1 TLV7031DBV

Commit message: Finished repeater schematic and updated resistor footprint
Parts:
- R1: footprint (none) -> CF12JT_Resistor_10_30_150_Ohms:STA_CF12_STP
- RR1: footprint CF12JT150R_Resistor_150:STA_CF12_STP -> CF12JT_Resistor_10_30_150_Ohms:STA_CF12_STP
Changed lines of the file:
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@@
 			)
 		)
-		(property "Footprint" "CF12JT150R_Resistor_150:STA_CF12_STP"
+		(property "Footprint" "CF12JT_Resistor_10_30_150_Ohms:STA_CF12_STP"
 			(at 133.096 67.056 90)
 			(hide yes)
@@
 			)
 		)
-		(property "Footprint" ""
+		(property "Footprint" "CF12JT_Resistor_10_30_150_Ohms:STA_CF12_STP"
 			(at 104.394 103.886 90)
 			(hide yes)

Commit message: Renamed the resistor footprints lol :3
Parts:
- R1, RR1: footprint CF12JT_Resistor_10_30_150_Ohms:STA_CF12_STP -> CF12JT_Resistor:STA_CF12_STP
- R2, R3, R4, R5, RD1, RD2, RD3, RD4: footprint CF12JT150R_Resistor_150:STA_CF12_STP -> CF12JT_Resistor:STA_CF12_STP
Changed lines of the file:
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@@
 			)
 		)
-		(property "Footprint" "CF12JT150R_Resistor_150:STA_CF12_STP"
+		(property "Footprint" "CF12JT_Resistor:STA_CF12_STP"
 			(at 193.294 84.074 90)
 			(hide yes)
@@
 			)
 		)
-		(property "Footprint" "CF12JT150R_Resistor_150:STA_CF12_STP"
+		(property "Footprint" "CF12JT_Resistor:STA_CF12_STP"
 			(at 193.294 103.124 90)
 			(hide yes)
@@
 			)
 		)
-		(property "Footprint" "CF12JT150R_Resistor_150:STA_CF12_STP"
+		(property "Footprint" "CF12JT_Resistor:STA_CF12_STP"
 			(at 193.294 65.024 90)
 			(hide yes)
@@
 			)
 		)
-		(property "Footprint" "CF12JT150R_Resistor_150:STA_CF12_STP"
+		(property "Footprint" "CF12JT_Resistor:STA_CF12_STP"
 			(at 135.636 117.856 90)
 			(hide yes)
@@
 			)
 		)
-		(property "Footprint" "CF12JT_Resistor_10_30_150_Ohms:STA_CF12_STP"
+		(property "Footprint" "CF12JT_Resistor:STA_CF12_STP"
 			(at 133.096 67.056 90)
 			(hide yes)
@@
 			)
 		)
-		(property "Footprint" "CF12JT150R_Resistor_150:STA_CF12_STP"
+		(property "Footprint" "CF12JT_Resistor:STA_CF12_STP"
 			(at 117.094 90.424 90)
 			(hide yes)
@@
 			)
 		)
-		(property "Footprint" "CF12JT_Resistor_10_30_150_Ohms:STA_CF12_STP"
+		(property "Footprint" "CF12JT_Resistor:STA_CF12_STP"
 			(at 104.394 103.886 90)
 			(hide yes)
@@
 			)
 		)
-		(property "Footprint" "CF12JT150R_Resistor_150:STA_CF12_STP"
+		(property "Footprint" "CF12JT_Resistor:STA_CF12_STP"
 			(at 136.144 90.424 90)
 			(hide yes)
@@
 			)
 		)
-		(property "Footprint" "CF12JT150R_Resistor_150:STA_CF12_STP"
+		(property "Footprint" "CF12JT_Resistor:STA_CF12_STP"
 			(at 117.094 115.824 90)
 			(hide yes)
@@
 			)
 		)
-		(property "Footprint" "CF12JT150R_Resistor_150:STA_CF12_STP"
+		(property "Footprint" "CF12JT_Resistor:STA_CF12_STP"
 			(at 193.294 122.174 90)
 			(hide yes)
