File: snapstone_pcb/skulk_sensor/skulk sensor.kicad_sch (KiCad schematic)
At the start: 8 parts, among them U1 ${SIM.PARAMS}

Commit message: did a bunch of stuff (something something Redstone Repeater PCB Changes)
Parts:
- C2: value 1uf -> 1 μF
- R2: value 2.2k -> 2.2 kΩ
Other:
- note added: "------->"
- note added: "MICROPHONE - BIAS"
- note added: "PEAK DETECTOR"
- note added: "PRE-AMPLIFIER"
- note added: "PUT VOLTAGE-TO-CURRENT THINGY HERE"
- note added: "this will cause a running period of 2.2ms, do we want a larger one? Just as a suggestion, what if we do 500μF * 1kΩ = 500ms ?"
- moved on the sheet: C2, C_OUT1, D1, R2, U1

Commit message: Updated resistor footprint project-wide
Parts:
- R1, R2: footprint (none) -> CF12JT_Resistor:STA_CF12_STP
Changed lines of the file:
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@@
 			)
 		)
-		(property "Footprint" ""
+		(property "Footprint" "CF12JT_Resistor:STA_CF12_STP"
 			(at 182.626 109.474 90)
 			(hide yes)
@@
 			)
 		)
-		(property "Footprint" ""
+		(property "Footprint" "CF12JT_Resistor:STA_CF12_STP"
 			(at 108.966 95.504 90)
 			(hide yes)
