File: snapstone_pcb/redstone_block/redstone_block.kicad_pcb (KiCad board)
At the start: 2 copper layers, 90 x 90 mm, 5 parts

Commit message: Made PCB for observer & redstone block!
Parts:
- added C_OUT2: ~, 691137710003_Board_To_Wire:691137710003_Board_To_Wire, F.Cu at (150.0, 133.0)
- added C_OUT3: ~, 691137710003_Board_To_Wire:691137710003_Board_To_Wire, F.Cu at (116.0, 100.0)
- added C_OUT4: ~, 691137710003_Board_To_Wire:691137710003_Board_To_Wire, F.Cu at (78.0, 104.9)
- R1: footprint CF12JT150R_Resistor_150:STA_CF12_STP -> CF12JT_Resistor:STA_CF12_STP
- moved C_OUT_LED1 60.3 mm to (120.0, 128.0), turned to 90 degrees
- moved R1 28.7 mm to (143.1, 91.0), turned to 0 degrees
- moved C_OUT_LED2 7.21 mm to (180.0, 128.0)
- moved C_OUT1 6.00 mm to (183.0, 100.0)
- moved BT1 4.12 mm to (150.0, 73.0), turned to 0 degrees
Connections:
- net Net-(C_OUT1-DAT) renamed OUT
- C_OUT_LED1 pad 2: unconnected-(C_OUT_LED1-GND-Pad2) -> GND
- C_OUT_LED2 pad 2: unconnected-(C_OUT_LED2-GND-Pad2) -> GND
Routing:
- net GND: track 72.1 -> 185.6 mm
- net VCC: track 98.9 -> 144.6 mm
- net OUT: track 162.3 -> 156.7 mm
Other:
- board size 90 x 90 mm -> 80 x 80 mm
- board text added: "Border of 3D Part"
- board text added: "Redstone Block Back"
- board text added: "Redstone Block Front"
- board text added: "We're cooked :з"
- board text removed: "DAT HERE"
